File: CRAMPS/CRAMPS.sch (KiCad schematic (older format))
At the start: 15 parts, among them M101 PCB_GREEN_RMC, M102 LOGO_OSHW, P101 SOCKET_6_LONG, P102 HEADER_2, P103 HEADER_2, P8 BB_EXP_CONN, P9 BB_EXP_CONN, Q101 2N7002K, SW101 SW_PUSH, SW102 SW_PUSH

Commit message: Fixed the pcb associations in the schematic
Parts:
- BB101: footprint BeagleBone-Pins -> beagleboneblack:BeagleBone-Pins
- LD101, LD102: footprint OSRAM-LED-0603 -> m_cramps:OSRAM-LED-0603
- M101: footprint OSHW_logo_2 -> RMC:OSHW_logo_2
- M102: footprint PCB_GREEN_RMC -> RMC:PCB_GREEN_RMC
- P101: footprint pin_strip_6 -> w_pin_strip:pin_strip_6
- P102, P103: footprint pin_strip_2 -> w_pin_strip:pin_strip_2
- P8, P9: footprint P8P9_PinHeader -> beagleboneblack:P8P9_PinHeader
- Q101: footprint SOT23GDS -> Tinkerforge:SOT23GDS
- R101, R102: footprint RESC1608x55N -> m_cramps:RESC1608x55N
- SW101, SW102: footprint SW_6x6_MULTI -> RMC:SW_6x6_MULTI
Changed lines of the file:
@@
 F 0 "M102" H 5250 7700 60  0000 C CNN
 F 1 "LOGO_OSHW" H 5250 7450 60  0000 C CNN
-F 2 "PCB_GREEN_RMC" H 5150 7600 60  0001 C CNN
+F 2 "RMC:PCB_GREEN_RMC" H 5150 7600 60  0001 C CNN
 F 3 "" H 5250 7550 60  0001 C CNN
 F 4 "N/A" H 5250 7550 60  0001 C CNN "Mfg"
@@
 F 0 "LD101" V 7075 5100 50  0000 C CNN
 F 1 "Yellow" V 7245 5100 50  0000 C CNN
-F 2 "OSRAM-LED-0603" H 7150 5100 60  0001 C CNN
+F 2 "m_cramps:OSRAM-LED-0603" H 7150 5100 60  0001 C CNN
 F 3 "" H 7150 5100 60  0001 C CNN
 F 4 "Osram" H 5500 6650 60  0001 C CNN "Mfg"
@@
 F 0 "M101" H 4350 7700 60  0000 C CNN
 F 1 "PCB_GREEN_RMC" H 4350 7450 60  0000 C CNN
-F 2 "OSHW_logo_2" H 4350 7550 60  0001 C CNN
+F 2 "RMC:OSHW_logo_2" H 4350 7550 60  0001 C CNN
 F 3 "" H 4350 7550 60  0000 C CNN
 F 4 "N/A" H 4350 7550 60  0001 C CNN "Mfg"
@@
 F 0 "SW102" H 9250 5850 50  0000 C CNN
 F 1 "SW_PUSH" H 9250 5620 50  0001 C CNN
-F 2 "SW_6x6_MULTI" H 9250 5700 60  0001 C CNN
+F 2 "RMC:SW_6x6_MULTI" H 9250 5700 60  0001 C CNN
 F 3 "" H 9250 5700 60  0001 C CNN
 F 4 "TE" H 5500 8550 60  0001 C CNN "Mfg"
@@
 F 0 "P103" H 9700 5850 60  0000 C CNN
 F 1 "HEADER_2" H 9700 5550 60  0001 C CNN
-F 2 "pin_strip_2" H 9650 5700 60  0001 C CNN
+F 2 "w_pin_strip:pin_strip_2" H 9650 5700 60  0001 C CNN
 F 3 "" H 9650 5700 60  0000 C CNN
 F 4 "Harwin" H 9650 5700 60  0001 C CNN "Mfg"
@@
 F 0 "SW101" H 9250 5050 50  0000 C CNN
 F 1 "SW_PUSH" H 9250 4820 50  0001 C CNN
-F 2 "SW_6x6_MULTI" H 9250 4900 60  0001 C CNN
+F 2 "RMC:SW_6x6_MULTI" H 9250 4900 60  0001 C CNN
 F 3 "" H 9250 4900 60  0001 C CNN
 F 4 "TE" H 5500 7750 60  0001 C CNN "Mfg"
@@
 F 0 "P102" H 9700 5050 60  0000 C CNN
 F 1 "HEADER_2" H 9700 4750 60  0001 C CNN
-F 2 "pin_strip_2" H 9650 4900 60  0001 C CNN
+F 2 "w_pin_strip:pin_strip_2" H 9650 4900 60  0001 C CNN
 F 3 "" H 9650 4900 60  0000 C CNN
 F 4 "Harwin" H 9650 4900 60  0001 C CNN "Mfg"
@@
 F 0 "R101" V 7100 4800 50  0000 C CNN
 F 1 "330R" V 7220 4800 50  0000 C CNN
-F 2 "RESC1608x55N" H 7150 4800 60  0001 C CNN
+F 2 "m_cramps:RESC1608x55N" H 7150 4800 60  0001 C CNN
 F 3 "" H 7150 4800 60  0000 C CNN
 F 4 "Stackpole" H 6450 5350 60  0001 C CNN "Mfg"
@@
 F 0 "Q101" H 7400 5600 70  0000 C CNN
 F 1 "2N7002K" H 7400 5500 60  0000 C CNN
-F 2 "SOT23GDS" H 7100 5550 60  0001 C CNN
+F 2 "Tinkerforge:SOT23GDS" H 7100 5550 60  0001 C CNN
 F 3 "" H 7100 5550 60  0000 C CNN
 F 4 "Diodes Inc." H 7100 5550 60  0001 C CNN "Mfg"
@@
 F 0 "LD102" V 8025 5100 50  0000 C CNN
 F 1 "Green" V 8195 5100 50  0000 C CNN
-F 2 "OSRAM-LED-0603" H 8100 5100 60  0001 C CNN
+F 2 "m_cramps:OSRAM-LED-0603" H 8100 5100 60  0001 C CNN
 F 3 "" H 8100 5100 60  0001 C CNN
 F 4 "Osram" H 6450 6650 60  0001 C CNN "Mfg"
@@
 F 0 "R102" V 8050 4800 50  0000 C CNN
 F 1 "330R" V 8170 4800 50  0000 C CNN
-F 2 "RESC1608x55N" H 8100 4800 60  0001 C CNN
+F 2 "m_cramps:RESC1608x55N" H 8100 4800 60  0001 C CNN
 F 3 "" H 8100 4800 60  0000 C CNN
 F 4 "Stackpole" H 6450 5350 60  0001 C CNN "Mfg"
@@
 F 0 "P8" H 3945 3355 60  0000 C CNN
 F 1 "BB_EXP_CONN" H 3950 885 60  0001 C CNN
-F 2 "P8P9_PinHeader" H 3600 900 60  0001 C CNN
+F 2 "beagleboneblack:P8P9_PinHeader" H 3600 900 60  0001 C CNN
 F 3 "" H 3600 900 60  0000 C CNN
 F 4 "Major League" H 3950 2100 60  0001 C CNN "Mfg"
@@
 F 0 "P9" H 3945 6155 60  0000 C CNN
 F 1 "BB_EXP_CONN" H 3950 3680 60  0001 C CNN
-F 2 "P8P9_PinHeader" H 3600 3700 60  0001 C CNN
+F 2 "beagleboneblack:P8P9_PinHeader" H 3600 3700 60  0001 C CNN
 F 3 "" H 3600 3700 60  0000 C CNN
 F 4 "Major League" H 3950 2100 60  0001 C CNN "Mfg"
@@
 F 0 "P101" H 1350 4600 60  0000 C CNN
 F 1 "SOCKET_6_LONG" H 1350 3900 60  0001 C CNN
-F 2 "pin_strip_6" H 1350 4250 60  0001 C CNN
+F 2 "w_pin_strip:pin_strip_6" H 1350 4250 60  0001 C CNN
 F 3 "" H 1350 4250 60  0000 C CNN
 F 4 "Sparkfun" H 1350 4250 60  0001 C CNN "Mfg"
@@
 F 0 "BB101" H 1525 6150 60  0000 C CNN
 F 1 "BeagleBone Black" H 1525 5200 60  0000 C CNN
-F 2 "BeagleBone-Pins" H 1425 6050 60  0001 C CNN
+F 2 "beagleboneblack:BeagleBone-Pins" H 1425 6050 60  0001 C CNN
 F 3 "" H 1250 5500 60  0000 C CNN
 F 4 "CircuitCo" H 1250 5500 60  0001 C CNN "Mfg"
