File: CRAMPS/con_inputs.sch (KiCad schematic (older format))
At the start: 34 parts, among them P501 HEADER_6, P502 HEADER_6X2, P503 HEADER_4X2, P504 HEADER_4X2, U501 74CBTD3861

Commit message: Updated schematic for new Kicad
Parts:
- P502: symbol HEADER_6X2 -> HEADER_6x2
- P503, P504: symbol HEADER_4X2 -> HEADER_4x2
- S501: symbol SHUNT -> Shunt
Changed lines of the file:
@@
 EESchema Schematic File Version 2
+LIBS:CRAMPS-rescue
 LIBS:power
 LIBS:m_cramps
@@
 LIBS:memory
 LIBS:xilinx
-LIBS:special
 LIBS:microcontrollers
 LIBS:dsp
@@
 LIBS:beagleboneblack
 LIBS:CRAMPS-cache
-EELAYER 27 0
+EELAYER 25 0
 EELAYER END
 $Descr A 11000 8500
@@
 SPI_CS0
 $Comp
-L HEADER_6X2 P502
+L HEADER_6x2 P502
 U 1 1 532C5F11
 P 1950 3750
@@
 $EndComp
 $Comp
-L HEADER_4X2 P504
+L HEADER_4x2 P504
 U 1 1 532C59EE
 P 6600 3200
@@
 Connection ~ 2400 2800
 $Comp
-L HEADER_4X2 P503
+L HEADER_4x2 P503
 U 1 1 535FE942
 P 1950 4450
@@
 	3100 4400 3700 4400
 $Comp
-L SHUNT S501
+L Shunt S501
 U 1 1 5361A40B
 P 9700 4350

Commit message: Fixed the pcb associations in the schematic
Parts:
- C501, C502, C503, C504, C505, C506, C507, C508, C509: footprint CAPC1608x55N -> m_cramps:CAPC1608x55N
- JP501: footprint pin_strip_2 -> w_pin_strip:pin_strip_2
- P501: footprint pin_strip_6 -> w_pin_strip:pin_strip_6
- P502: footprint pin_strip_6x2 -> w_pin_strip:pin_strip_6x2
- P503, P504: footprint pin_strip_4x2 -> w_pin_strip:pin_strip_4x2
- R501, R502, R503, R504, R505, R506, R507, R508, R509, R510, R511, R512, R513, R514, R515, R516, R517, R518: footprint RESC1608x55N -> m_cramps:RESC1608x55N
- S501: footprint Shunt -> m_cramps:Shunt
- U501: footprint SOIC127P1030X265-24N -> m_cramps:SOIC127P1030X265-24N
Changed lines of the file:
@@
 F 0 "C501" H 3850 2460 50  0000 L CNN
 F 1 "100n" H 3850 2390 50  0000 L CNN
-F 2 "CAPC1608x55N" H 3800 2450 60  0001 C CNN
+F 2 "m_cramps:CAPC1608x55N" H 3800 2450 60  0001 C CNN
 F 3 "" H 3800 2450 60  0001 C CNN
 F 4 "Murata" H 5150 6500 60  0001 C CNN "Mfg"
@@
 F 0 "P502" H 1950 4100 60  0000 C CNN
 F 1 "HEADER_6X2" H 1950 3400 60  0001 C CNN
-F 2 "pin_strip_6x2" H 1950 3750 60  0001 C CNN
+F 2 "w_pin_strip:pin_strip_6x2" H 1950 3750 60  0001 C CNN
 F 3 "" H 1950 3750 60  0000 C CNN
 F 4 "Harwin" H 1950 3750 60  0001 C CNN "Mfg"
@@
 F 0 "P501" H 1650 4100 60  0000 C CNN
 F 1 "HEADER_6" H 1600 3400 60  0001 C CNN
-F 2 "pin_strip_6" H 1600 3750 60  0001 C CNN
+F 2 "w_pin_strip:pin_strip_6" H 1600 3750 60  0001 C CNN
 F 3 "" H 1600 3750 60  0000 C CNN
 F 4 "Harwin" H 9500 5350 60  0001 C CNN "Mfg"
@@
 F 0 "C502" H 8050 2135 50  0000 L CNN
 F 1 "100n" H 8050 2065 50  0000 L CNN
-F 2 "CAPC1608x55N" H 8000 2100 60  0001 C CNN
+F 2 "m_cramps:CAPC1608x55N" H 8000 2100 60  0001 C CNN
 F 3 "" H 8000 2100 60  0001 C CNN
 F 4 "Murata" H 9050 6750 60  0001 C CNN "Mfg"
@@
 F 0 "C503" H 8050 3010 50  0000 L CNN
 F 1 "100n" H 8050 2940 50  0000 L CNN
-F 2 "CAPC1608x55N" H 8000 3000 60  0001 C CNN
+F 2 "m_cramps:CAPC1608x55N" H 8000 3000 60  0001 C CNN
 F 3 "" H 8000 3000 60  0001 C CNN
 F 4 "Murata" H 9050 6050 60  0001 C CNN "Mfg"
@@
 F 0 "C504" H 8050 3910 50  0000 L CNN
 F 1 "100n" H 8050 3840 50  0000 L CNN
-F 2 "CAPC1608x55N" H 8000 3900 60  0001 C CNN
+F 2 "m_cramps:CAPC1608x55N" H 8000 3900 60  0001 C CNN
 F 3 "" H 8000 3900 60  0001 C CNN
 F 4 "Murata" H 9050 5350 60  0001 C CNN "Mfg"
@@
 F 0 "C505" H 8050 4810 50  0000 L CNN
 F 1 "100n" H 8050 4740 50  0000 L CNN
-F 2 "CAPC1608x55N" H 8000 4800 60  0001 C CNN
+F 2 "m_cramps:CAPC1608x55N" H 8000 4800 60  0001 C CNN
 F 3 "" H 8000 4800 60  0001 C CNN
 F 4 "Murata" H 9050 4650 60  0001 C CNN "Mfg"
@@
 F 0 "C509" H 8450 4810 50  0000 L CNN
 F 1 "10u" H 8450 4740 50  0000 L CNN
-F 2 "CAPC1608x55N" H 8400 4800 60  0001 C CNN
+F 2 "m_cramps:CAPC1608x55N" H 8400 4800 60  0001 C CNN
 F 3 "" H 8400 4800 60  0001 C CNN
 F 4 "Taiyo Yuden" H 9050 4650 60  0001 C CNN "Mfg"
@@
 F 0 "C508" H 8450 3910 50  0000 L CNN
 F 1 "10u" H 8450 3840 50  0000 L CNN
-F 2 "CAPC1608x55N" H 8400 3900 60  0001 C CNN
+F 2 "m_cramps:CAPC1608x55N" H 8400 3900 60  0001 C CNN
 F 3 "" H 8400 3900 60  0001 C CNN
 F 4 "Taiyo Yuden" H 9050 5350 60  0001 C CNN "Mfg"
@@
 F 0 "C507" H 8450 3010 50  0000 L CNN
 F 1 "10u" H 8450 2940 50  0000 L CNN
-F 2 "CAPC1608x55N" H 8400 3000 60  0001 C CNN
+F 2 "m_cramps:CAPC1608x55N" H 8400 3000 60  0001 C CNN
 F 3 "" H 8400 3000 60  0001 C CNN
 F 4 "Taiyo Yuden" H 9050 6050 60  0001 C CNN "Mfg"
@@
 F 0 "C506" H 8450 2110 50  0000 L CNN
 F 1 "10u" H 8450 2040 50  0000 L CNN
-F 2 "CAPC1608x55N" H 8400 2100 60  0001 C CNN
+F 2 "m_cramps:CAPC1608x55N" H 8400 2100 60  0001 C CNN
 F 3 "" H 8400 2100 60  0001 C CNN
 F 4 "Taiyo Yuden" H 9050 6750 60  0001 C CNN "Mfg"
@@
 F 0 "JP501" H 8850 4325 60  0000 C CNN
 F 1 "HEADER_2" H 8875 4575 60  0001 C CNN
-F 2 "pin_strip_2" H 8850 4400 60  0001 C CNN
+F 2 "w_pin_strip:pin_strip_2" H 8850 4400 60  0001 C CNN
 F 3 "" H 8850 4400 60  0000 C CNN
 F 4 "Harwin" H 9150 4850 60  0001 C CNN "Mfg"
@@
 F 0 "R515" V 7650 1900 50  0000 C CNN
 F 1 "4k7" V 7770 1900 50  0000 C CNN
-F 2 "RESC1608x55N" H 7700 1900 60  0001 C CNN
+F 2 "m_cramps:RESC1608x55N" H 7700 1900 60  0001 C CNN
 F 3 "" H 7700 1900 60  0001 C CNN
 F 4 "Stackpole" H 11250 4100 60  0001 C CNN "Mfg"
@@
 F 0 "R516" V 7650 2800 50  0000 C CNN
 F 1 "4k7" V 7770 2800 50  0000 C CNN
-F 2 "RESC1608x55N" H 7700 2800 60  0001 C CNN
+F 2 "m_cramps:RESC1608x55N" H 7700 2800 60  0001 C CNN
 F 3 "" H 7700 2800 60  0001 C CNN
 F 4 "Stackpole" H 11250 5000 60  0001 C CNN "Mfg"
@@
 F 0 "R517" V 7650 3700 50  0000 C CNN
 F 1 "4k7" V 7770 3700 50  0000 C CNN
-F 2 "RESC1608x55N" H 7700 3700 60  0001 C CNN
+F 2 "m_cramps:RESC1608x55N" H 7700 3700 60  0001 C CNN
 F 3 "" H 7700 3700 60  0001 C CNN
 F 4 "Stackpole" H 11250 5900 60  0001 C CNN "Mfg"
@@
 F 0 "R518" V 7650 4600 50  0000 C CNN
 F 1 "4k7" V 7770 4600 50  0000 C CNN
-F 2 "RESC1608x55N" H 7700 4600 60  0001 C CNN
+F 2 "m_cramps:RESC1608x55N" H 7700 4600 60  0001 C CNN
 F 3 "" H 7700 4600 60  0001 C CNN
 F 4 "Stackpole" H 11250 6800 60  0001 C CNN "Mfg"
@@
 F 0 "R511" V 7350 1700 50  0000 C CNN
 F 1 "2K0 1%" V 7470 1700 50  0000 C CNN
-F 2 "RESC1608x55N" H 7400 1700 60  0001 C CNN
+F 2 "m_cramps:RESC1608x55N" H 7400 1700 60  0001 C CNN
 F 3 "" H 7400 1700 60  0001 C CNN
 F 4 "Stackpole" H 10950 3900 60  0001 C CNN "Mfg"
@@
 F 0 "R512" V 7350 2600 50  0000 C CNN
 F 1 "2K0 1%" V 7470 2600 50  0000 C CNN
-F 2 "RESC1608x55N" H 7400 2600 60  0001 C CNN
+F 2 "m_cramps:RESC1608x55N" H 7400 2600 60  0001 C CNN
 F 3 "" H 7400 2600 60  0001 C CNN
 F 4 "Stackpole" H 10950 3900 60  0001 C CNN "Mfg"
@@
 F 0 "R513" V 7350 3500 50  0000 C CNN
 F 1 "2K0 1%" V 7470 3500 50  0000 C CNN
-F 2 "RESC1608x55N" H 7400 3500 60  0001 C CNN
+F 2 "m_cramps:RESC1608x55N" H 7400 3500 60  0001 C CNN
 F 3 "" H 7400 3500 60  0001 C CNN
 F 4 "Stackpole" H 10950 3900 60  0001 C CNN "Mfg"
@@
 F 0 "R514" V 7350 4400 50  0000 C CNN
 F 1 "2K0 1%" V 7470 4400 50  0000 C CNN
-F 2 "RESC1608x55N" H 7400 4400 60  0001 C CNN
+F 2 "m_cramps:RESC1608x55N" H 7400 4400 60  0001 C CNN
 F 3 "" H 7400 4400 60  0001 C CNN
 F 4 "Stackpole" H 10950 3900 60  0001 C CNN "Mfg"
@@
 F 0 "P504" H 6600 3450 60  0000 C CNN
 F 1 "HEADER_4X2" H 6600 2950 60  0001 C CNN
-F 2 "pin_strip_4x2" H 6600 3200 60  0001 C CNN
+F 2 "w_pin_strip:pin_strip_4x2" H 6600 3200 60  0001 C CNN
 F 3 "" H 6600 3200 60  0000 C CNN
 F 4 "Harwin" H 7050 5350 60  0001 C CNN "Mfg"
@@
 F 0 "U501" H 4300 4600 60  0000 L CNN
 F 1 "74CBTD3861" H 4220 3385 60  0000 L CNN
-F 2 "SOIC127P1030X265-24N" H 4200 4100 60  0001 C CNN
+F 2 "m_cramps:SOIC127P1030X265-24N" H 4200 4100 60  0001 C CNN
 F 3 "" H 4200 4100 60  0000 C CNN
 F 4 "TI" H 4200 4000 60  0001 C CNN "Mfg"
@@
 F 0 "R501" V 2250 3000 50  0000 C CNN
 F 1 "10k" V 2370 3000 50  0000 C CNN
-F 2 "RESC1608x55N" H 2300 3000 60  0001 C CNN
+F 2 "m_cramps:RESC1608x55N" H 2300 3000 60  0001 C CNN
 F 3 "" H 2300 3000 60  0001 C CNN
 F 4 "Stackpole" H 3650 7500 60  0001 C CNN "Mfg"
@@
 F 0 "R502" V 2350 3200 50  0000 C CNN
 F 1 "10k" V 2470 3200 50  0000 C CNN
-F 2 "RESC1608x55N" H 2400 3200 60  0001 C CNN
+F 2 "m_cramps:RESC1608x55N" H 2400 3200 60  0001 C CNN
 F 3 "" H 2400 3200 60  0001 C CNN
 F 4 "Stackpole" H 3750 7700 60  0001 C CNN "Mfg"
@@
 F 0 "R503" V 2450 3000 50  0000 C CNN
 F 1 "10k" V 2570 3000 50  0000 C CNN
-F 2 "RESC1608x55N" H 2500 3000 60  0001 C CNN
+F 2 "m_cramps:RESC1608x55N" H 2500 3000 60  0001 C CNN
 F 3 "" H 2500 3000 60  0001 C CNN
 F 4 "Stackpole" H 3850 7500 60  0001 C CNN "Mfg"
@@
 F 0 "R504" V 2550 3200 50  0000 C CNN
 F 1 "10k" V 2670 3200 50  0000 C CNN
-F 2 "RESC1608x55N" H 2600 3200 60  0001 C CNN
+F 2 "m_cramps:RESC1608x55N" H 2600 3200 60  0001 C CNN
 F 3 "" H 2600 3200 60  0001 C CNN
 F 4 "Stackpole" H 3950 7700 60  0001 C CNN "Mfg"
@@
 F 0 "R505" V 2650 3000 50  0000 C CNN
 F 1 "10k" V 2770 3000 50  0000 C CNN
-F 2 "RESC1608x55N" H 2700 3000 60  0001 C CNN
+F 2 "m_cramps:RESC1608x55N" H 2700 3000 60  0001 C CNN
 F 3 "" H 2700 3000 60  0001 C CNN
 F 4 "Stackpole" H 4050 7500 60  0001 C CNN "Mfg"
@@
 F 0 "R506" V 2750 3200 50  0000 C CNN
 F 1 "10k" V 2870 3200 50  0000 C CNN
-F 2 "RESC1608x55N" H 2800 3200 60  0001 C CNN
+F 2 "m_cramps:RESC1608x55N" H 2800 3200 60  0001 C CNN
 F 3 "" H 2800 3200 60  0001 C CNN
 F 4 "Stackpole" H 4150 7700 60  0001 C CNN "Mfg"
@@
 F 0 "R507" V 2850 3000 50  0000 C CNN
 F 1 "10k" V 2970 3000 50  0000 C CNN
-F 2 "RESC1608x55N" H 2900 3000 60  0001 C CNN
+F 2 "m_cramps:RESC1608x55N" H 2900 3000 60  0001 C CNN
 F 3 "" H 2900 3000 60  0001 C CNN
 F 4 "Stackpole" H 4250 7500 60  0001 C CNN "Mfg"
@@
 F 0 "R508" V 2950 3200 50  0000 C CNN
 F 1 "10k" V 3070 3200 50  0000 C CNN
-F 2 "RESC1608x55N" H 3000 3200 60  0001 C CNN
+F 2 "m_cramps:RESC1608x55N" H 3000 3200 60  0001 C CNN
 F 3 "" H 3000 3200 60  0001 C CNN
 F 4 "Stackpole" H 4350 7700 60  0001 C CNN "Mfg"
@@
 F 0 "R509" V 3050 3000 50  0000 C CNN
 F 1 "10k" V 3170 3000 50  0000 C CNN
-F 2 "RESC1608x55N" H 3100 3000 60  0001 C CNN
+F 2 "m_cramps:RESC1608x55N" H 3100 3000 60  0001 C CNN
 F 3 "" H 3100 3000 60  0001 C CNN
 F 4 "Stackpole" H 4450 7500 60  0001 C CNN "Mfg"
@@
 F 0 "R510" V 3150 3200 50  0000 C CNN
 F 1 "10k" V 3270 3200 50  0000 C CNN
-F 2 "RESC1608x55N" H 3200 3200 60  0001 C CNN
+F 2 "m_cramps:RESC1608x55N" H 3200 3200 60  0001 C CNN
 F 3 "" H 3200 3200 60  0001 C CNN
 F 4 "Stackpole" H 4550 7700 60  0001 C CNN "Mfg"
@@
 F 0 "P503" H 1950 4700 60  0000 C CNN
 F 1 "HEADER_4X2" H 1950 4200 60  0001 C CNN
-F 2 "pin_strip_4x2" H 1950 4450 60  0001 C CNN
+F 2 "w_pin_strip:pin_strip_4x2" H 1950 4450 60  0001 C CNN
 F 3 "" H 1950 4450 60  0000 C CNN
 F 4 "Harwin" H 7050 5350 60  0001 C CNN "Mfg"
@@
 F 0 "S501" H 9700 4450 60  0000 C CNN
 F 1 "SHUNT" H 9700 4250 60  0000 C CNN
-F 2 "Shunt" H 9700 4350 60  0001 C CNN
+F 2 "m_cramps:Shunt" H 9700 4350 60  0001 C CNN
 F 3 "" H 9700 4350 60  0000 C CNN
 F 4 "TE" H 9200 2450 60  0001 C CNN "Mfg"
