File: CRAMPS/con_outputs.sch (KiCad schematic (older format))
At the start: 50 parts, among them P401 PT_2,5-2-5,0-H, P402 PT_2,5-2-5,0-H, P403 PT_2,5-2-5,0-H, P404 PT_1,5-3-3,5-H, P405 PT_1,5-2-3,5-H, P406 PT_1,5-2-3,5-H, P407 KK-2.54-2W, P408 PT_1,5-2-3,5-H, P409 KK-2.54-2W, Q401 IRLB8743PBF, Q402 IRLB8743PBF, Q403 IRLB8743PBF, Q404 DMN2075U, Q405 IRLB8743PBF, Q406 DMN2075U

Commit message: Updated schematic for new Kicad
Parts:
- C401: symbol CP1 -> CP1-RESCUE-CRAMPS
Changed lines of the file:
@@
 EESchema Schematic File Version 2
+LIBS:CRAMPS-rescue
 LIBS:power
 LIBS:m_cramps
@@
 LIBS:memory
 LIBS:xilinx
-LIBS:special
 LIBS:microcontrollers
 LIBS:dsp
@@
 LIBS:beagleboneblack
 LIBS:CRAMPS-cache
-EELAYER 27 0
+EELAYER 25 0
 EELAYER END
 $Descr A 11000 8500
@@
 Ext_Pwr
 $Comp
-L CP1 C401
+L CP1-RESCUE-CRAMPS C401
 U 1 1 533060BF
 P 2900 5050

Commit message: Fixed the pcb associations in the schematic
Parts:
- C401: footprint c_elec_6.3x7.7 -> Capacitors_SMD:c_elec_6.3x7.7
- C402, C403, C404, C405, C406, C407: footprint CAPC1608x55N -> m_cramps:CAPC1608x55N
- D401, D402, D403, D404, D405, D406: footprint DIOM5127X229N -> m_cramps:DIOM5127X229N
- F401, F402: footprint Fuse-Loose -> m_cramps:Fuse-Loose
- FH401, FH402: footprint Keystone-3568 -> m_cramps:Keystone-3568
- LD401, LD402, LD403, LD404, LD405, LD406: footprint OSRAM-LED-0603 -> m_cramps:OSRAM-LED-0603
- P401, P402, P403: footprint PT_2,5-2-5,0-H -> m_cramps:PT_2,5-2-5,0-H
- P404: footprint PT_1,5-3-3,5-H -> m_cramps:PT_1,5-3-3,5-H
- P405, P406, P408: footprint PT_1,5-2-3,5-H -> m_cramps:PT_1,5-2-3,5-H
- P407, P409: footprint CONN_KK_2.54_2W -> RMC:CONN_KK_2.54_2W
- Q401, Q402, Q403, Q405: footprint TO-220AB_IRF2804_RMC -> RMC:TO-220AB_IRF2804_RMC
- Q404, Q406: footprint SOT23GDS -> Tinkerforge:SOT23GDS
- R401, R402, R403, R404, R405, R406, R407, R408, R409, R410, R411, R412: footprint RESC1608x55N -> m_cramps:RESC1608x55N
