File: CRAMPS/e-stop.sch (KiCad schematic (older format))
At the start: 34 parts, among them P301 HEADER_2, P302 KK-2.54-2W, P303 HEADER_4X2, P304 HEADER_3X2, P305 HEADER_6, Q301 2N7002K, Q302 2N7002K, Q303 2N7002K, Q304 2N7002K, Q305 2N7002K, U301 24C256, U302 74ACT244

Commit message: Updated schematic for new Kicad
Parts:
- JP301: symbol HEADER_2X2 -> HEADER_2x2
- P303: symbol HEADER_4X2 -> HEADER_4x2
- P304: symbol HEADER_3X2 -> HEADER_3x2
- S301: symbol SHUNT -> Shunt
Changed lines of the file:
@@
 EESchema Schematic File Version 2
+LIBS:CRAMPS-rescue
 LIBS:power
 LIBS:m_cramps
@@
 LIBS:memory
 LIBS:xilinx
-LIBS:special
 LIBS:microcontrollers
 LIBS:dsp
@@
 LIBS:beagleboneblack
 LIBS:CRAMPS-cache
-EELAYER 27 0
+EELAYER 25 0
 EELAYER END
 $Descr A 11000 8500
@@
 Address and WP pins have internal pull-down\nDefault configuration is no shunts populated:\nAddr = 0xA8\nWP = Disabled (writes allowed)
 $Comp
-L HEADER_2X2 JP301
+L HEADER_2x2 JP301
 U 1 1 53319970
 P 1950 6750
@@
 $EndComp
 $Comp
-L HEADER_4X2 P303
+L HEADER_4x2 P303
 U 1 1 53319778
 P 7050 5250
@@
 	6900 5200 6700 5200
 $Comp
-L HEADER_3X2 P304
+L HEADER_3x2 P304
 U 1 1 535FF544
 P 7050 6200
@@
 	1600 4200 1600 4300
 $Comp
-L SHUNT S301
+L Shunt S301
 U 1 1 536179A3
 P 4200 5050

Commit message: Fixed the pcb associations in the schematic
Parts:
- C301, C302: footprint CAPC1608x55N -> m_cramps:CAPC1608x55N
- JP301: footprint pin_strip_2x2 -> w_pin_strip:pin_strip_2x2
- LD301, LD302: footprint OSRAM-LED-0603 -> m_cramps:OSRAM-LED-0603
- P301: footprint pin_strip_2 -> w_pin_strip:pin_strip_2
- P302: footprint CONN_KK_2.54_2W -> RMC:CONN_KK_2.54_2W
- P303: footprint pin_strip_4x2 -> w_pin_strip:pin_strip_4x2
- P304: footprint pin_strip_3x2 -> w_pin_strip:pin_strip_3x2
- P305: footprint pin_strip_6 -> w_pin_strip:pin_strip_6
- Q301, Q302, Q303, Q304, Q305: footprint SOT23GDS -> Tinkerforge:SOT23GDS
- R301, R302, R303, R304, R305, R306, R307, R308, R309, R310, R311, R312, R313, R314, R315, R316: footprint RESC1608x55N -> m_cramps:RESC1608x55N
- S301: footprint Shunt -> m_cramps:Shunt
- U301: footprint SOIC127P600X175-8AN -> m_cramps:SOIC127P600X175-8AN
- U302: footprint SOIC127P1032X265-20N -> m_cramps:SOIC127P1032X265-20N
Changed lines of the file:
@@
 F 0 "C302" H 5850 1210 50  0000 L CNN
 F 1 "100n" H 5850 1140 50  0000 L CNN
-F 2 "CAPC1608x55N" H 5800 1200 60  0001 C CNN
+F 2 "m_cramps:CAPC1608x55N" H 5800 1200 60  0001 C CNN
 F 3 "" H 5800 1200 60  0001 C CNN
 F 4 "Murata" H 1950 6450 60  0001 C CNN "Mfg"
@@
 F 0 "LD302" V 3125 3300 50  0000 C CNN
 F 1 "Red" V 3295 3300 50  0000 C CNN
-F 2 "OSRAM-LED-0603" H 3200 3300 60  0001 C CNN
+F 2 "m_cramps:OSRAM-LED-0603" H 3200 3300 60  0001 C CNN
 F 3 "" H 3200 3300 60  0001 C CNN
 F 4 "Osram" H 1550 4850 60  0001 C CNN "Mfg"
@@
 F 0 "R305" V 3150 3000 50  0000 C CNN
 F 1 "220R" V 3270 3000 50  0000 C CNN
-F 2 "RESC1608x55N" H 3200 3000 60  0001 C CNN
+F 2 "m_cramps:RESC1608x55N" H 3200 3000 60  0001 C CNN
 F 3 "" H 3200 3000 60  0000 C CNN
 F 4 "Stackpole" H 6250 5550 60  0001 C CNN "Mfg"
@@
 F 0 "Q303" H 1950 5000 70  0000 C CNN
 F 1 "2N7002K" H 1900 4650 60  0000 C CNN
-F 2 "SOT23GDS" H 2150 4850 60  0001 C CNN
+F 2 "Tinkerforge:SOT23GDS" H 2150 4850 60  0001 C CNN
 F 3 "" H 2150 4850 60  0000 C CNN
 F 4 "Diodes Inc." H 7100 5950 60  0001 C CNN "Mfg"
@@
 F 0 "Q302" H 1900 2550 70  0000 C CNN
 F 1 "2N7002K" H 1850 2200 60  0000 C CNN
-F 2 "SOT23GDS" H 2100 2400 60  0001 C CNN
+F 2 "Tinkerforge:SOT23GDS" H 2100 2400 60  0001 C CNN
 F 3 "" H 2100 2400 60  0000 C CNN
 F 4 "Diodes Inc." H 7100 5550 60  0001 C CNN "Mfg"
@@
 F 0 "Q304" H 2300 2550 70  0000 C CNN
 F 1 "2N7002K" H 2250 2200 60  0000 C CNN
-F 2 "SOT23GDS" H 2500 2400 60  0001 C CNN
+F 2 "Tinkerforge:SOT23GDS" H 2500 2400 60  0001 C CNN
 F 3 "" H 2500 2400 60  0000 C CNN
 F 4 "Diodes Inc." H 7100 5550 60  0001 C CNN "Mfg"
@@
 F 0 "P302" H 2050 3900 60  0000 C CNN
 F 1 "KK-2.54-2W" H 2050 3580 60  0001 C CNN
-F 2 "CONN_KK_2.54_2W" H 2000 3750 60  0001 C CNN
+F 2 "RMC:CONN_KK_2.54_2W" H 2000 3750 60  0001 C CNN
 F 3 "" H 2000 3750 60  0000 C CNN
 F 4 "Molex" H 2000 3750 60  0001 C CNN "Mfg"
@@
 F 0 "R304" V 2550 3500 50  0000 C CNN
 F 1 "4k7" V 2670 3500 50  0000 C CNN
-F 2 "RESC1608x55N" H 2600 3500 60  0001 C CNN
+F 2 "m_cramps:RESC1608x55N" H 2600 3500 60  0001 C CNN
 F 3 "" H 2600 3500 60  0001 C CNN
 F 4 "Stackpole" H 6150 5700 60  0001 C CNN "Mfg"
@@
 F 0 "LD301" V 2375 1750 50  0000 C CNN
 F 1 "Green" V 2545 1750 50  0000 C CNN
-F 2 "OSRAM-LED-0603" H 2450 1750 60  0001 C CNN
+F 2 "m_cramps:OSRAM-LED-0603" H 2450 1750 60  0001 C CNN
 F 3 "" H 2450 1750 60  0001 C CNN
 F 4 "Osram" H 800 3300 60  0001 C CNN "Mfg"
@@
 F 0 "R303" V 2400 1400 50  0000 C CNN
 F 1 "330R" V 2520 1400 50  0000 C CNN
-F 2 "RESC1608x55N" H 2450 1400 60  0001 C CNN
+F 2 "m_cramps:RESC1608x55N" H 2450 1400 60  0001 C CNN
 F 3 "" H 2450 1400 60  0000 C CNN
 F 4 "Stackpole" H 6450 5350 60  0001 C CNN "Mfg"
@@
 F 0 "Q301" H 1350 5000 70  0000 C CNN
 F 1 "2N7002K" H 1300 4650 60  0000 C CNN
-F 2 "SOT23GDS" H 1550 4850 60  0001 C CNN
+F 2 "Tinkerforge:SOT23GDS" H 1550 4850 60  0001 C CNN
 F 3 "" H 1550 4850 60  0000 C CNN
 F 4 "Diodes Inc." H 7100 5950 60  0001 C CNN "Mfg"
@@
 F 0 "U302" H 5950 3250 60  0000 C CNN
 F 1 "74ACT244" V 5800 2600 60  0000 C CNN
-F 2 "SOIC127P1032X265-20N" H 5800 2600 60  0001 C CNN
+F 2 "m_cramps:SOIC127P1032X265-20N" H 5800 2600 60  0001 C CNN
 F 3 "" H 5800 2600 60  0000 C CNN
 F 4 "Fairchild" H 5800 2600 60  0001 C CNN "Mfg"
@@
 F 0 "C301" H 1450 7135 50  0000 L CNN
 F 1 "100n" H 1450 7065 50  0000 L CNN
-F 2 "CAPC1608x55N" H 1438 6950 30  0001 C CNN
+F 2 "m_cramps:CAPC1608x55N" H 1438 6950 30  0001 C CNN
 F 3 "" H 1400 7100 60  0000 C CNN
 F 4 "Murata" H 1650 7350 60  0001 C CNN "Mfg"
@@
 F 0 "JP301" H 1950 6900 60  0000 C CNN
 F 1 "HEADER_2X2" H 1950 6600 60  0001 C CNN
-F 2 "pin_strip_2x2" H 1950 6750 60  0001 C CNN
+F 2 "w_pin_strip:pin_strip_2x2" H 1950 6750 60  0001 C CNN
 F 3 "" H 1950 6750 60  0000 C CNN
 F 4 "Harwin" H 1950 6750 60  0001 C CNN "Mfg"
@@
 F 0 "U301" H 2900 7450 60  0000 C CNN
 F 1 "24C256" H 2750 7100 60  0000 C CNN
-F 2 "SOIC127P600X175-8AN" H 2750 7100 60  0001 C CNN
+F 2 "m_cramps:SOIC127P600X175-8AN" H 2750 7100 60  0001 C CNN
 F 3 "" H 2750 7100 60  0000 C CNN
 F 4 "On Semi" H 2750 7100 60  0001 C CNN "Mfg"
@@
 F 0 "P305" H 9500 5700 60  0000 C CNN
 F 1 "HEADER_6" H 9500 5000 60  0001 C CNN
-F 2 "pin_strip_6" H 9500 5350 60  0001 C CNN
+F 2 "w_pin_strip:pin_strip_6" H 9500 5350 60  0001 C CNN
 F 3 "" H 9500 5350 60  0000 C CNN
 F 4 "Harwin" H 9500 5350 60  0001 C CNN "Mfg"
@@
 F 0 "P303" H 7050 5500 60  0000 C CNN
 F 1 "HEADER_4X2" H 7050 5000 60  0001 C CNN
-F 2 "pin_strip_4x2" H 7050 5250 60  0001 C CNN
+F 2 "w_pin_strip:pin_strip_4x2" H 7050 5250 60  0001 C CNN
 F 3 "" H 7050 5250 60  0000 C CNN
 F 4 "Harwin" H 7050 5250 60  0001 C CNN "Mfg"
@@
 F 0 "P301" H 1350 2100 60  0000 C CNN
 F 1 "HEADER_2" H 1350 1780 60  0001 C CNN
-F 2 "pin_strip_2" H 1300 1950 60  0001 C CNN
+F 2 "w_pin_strip:pin_strip_2" H 1300 1950 60  0001 C CNN
 F 3 "" H 1300 1950 60  0000 C CNN
 F 4 "Harwin" H 1300 1950 60  0001 C CNN "Mfg"
@@
 F 0 "R302" V 1450 2800 50  0000 C CNN
 F 1 "2K7" V 1570 2800 50  0000 C CNN
-F 2 "RESC1608x55N" H 1500 2800 60  0001 C CNN
+F 2 "m_cramps:RESC1608x55N" H 1500 2800 60  0001 C CNN
 F 3 "" H 1500 2800 60  0000 C CNN
 F 4 "Stackpole" H 5950 5350 60  0001 C CNN "Mfg"
@@
 F 0 "R301" V 1550 4400 50  0000 C CNN
 F 1 "10k" V 1670 4400 50  0000 C CNN
-F 2 "RESC1608x55N" H 1600 4400 60  0001 C CNN
+F 2 "m_cramps:RESC1608x55N" H 1600 4400 60  0001 C CNN
 F 3 "" H 1600 4400 60  0001 C CNN
 F 4 "Stackpole" H 2950 8900 60  0001 C CNN "Mfg"
@@
 F 0 "R314" V 6650 1800 50  0000 C CNN
 F 1 "4k7" V 6770 1800 50  0000 C CNN
-F 2 "RESC1608x55N" H 6700 1800 60  0001 C CNN
+F 2 "m_cramps:RESC1608x55N" H 6700 1800 60  0001 C CNN
 F 3 "" H 6700 1800 60  0001 C CNN
 F 4 "Stackpole" H 10250 4000 60  0001 C CNN "Mfg"
@@
 F 0 "R310" V 6350 1800 50  0000 C CNN
 F 1 "10k" V 6470 1800 50  0000 C CNN
-F 2 "RESC1608x55N" H 6400 1800 60  0001 C CNN
+F 2 "m_cramps:RESC1608x55N" H 6400 1800 60  0001 C CNN
 F 3 "" H 6400 1800 60  0001 C CNN
 F 4 "Stackpole" H 7750 6300 60  0001 C CNN "Mfg"
@@
 F 0 "R309" V 6250 3300 50  0000 C CNN
 F 1 "10k" V 6370 3300 50  0000 C CNN
-F 2 "RESC1608x55N" H 6300 3300 60  0001 C CNN
+F 2 "m_cramps:RESC1608x55N" H 6300 3300 60  0001 C CNN
 F 3 "" H 6300 3300 60  0001 C CNN
 F 4 "Stackpole" H 7650 7800 60  0001 C CNN "Mfg"
@@
 F 0 "R311" V 6350 3500 50  0000 C CNN
 F 1 "10k" V 6470 3500 50  0000 C CNN
-F 2 "RESC1608x55N" H 6400 3500 60  0001 C CNN
+F 2 "m_cramps:RESC1608x55N" H 6400 3500 60  0001 C CNN
 F 3 "" H 6400 3500 60  0001 C CNN
 F 4 "Stackpole" H 7750 8000 60  0001 C CNN "Mfg"
@@
 F 0 "R312" V 6450 3300 50  0000 C CNN
 F 1 "10k" V 6570 3300 50  0000 C CNN
-F 2 "RESC1608x55N" H 6500 3300 60  0001 C CNN
+F 2 "m_cramps:RESC1608x55N" H 6500 3300 60  0001 C CNN
 F 3 "" H 6500 3300 60  0001 C CNN
 F 4 "Stackpole" H 7850 7800 60  0001 C CNN "Mfg"
@@
 F 0 "R313" V 6550 3500 50  0000 C CNN
 F 1 "10k" V 6670 3500 50  0000 C CNN
-F 2 "RESC1608x55N" H 6600 3500 60  0001 C CNN
+F 2 "m_cramps:RESC1608x55N" H 6600 3500 60  0001 C CNN
 F 3 "" H 6600 3500 60  0001 C CNN
 F 4 "Stackpole" H 7950 8000 60  0001 C CNN "Mfg"
@@
 F 0 "R315" V 6650 3300 50  0000 C CNN
 F 1 "10k" V 6770 3300 50  0000 C CNN
-F 2 "RESC1608x55N" H 6700 3300 60  0001 C CNN
+F 2 "m_cramps:RESC1608x55N" H 6700 3300 60  0001 C CNN
 F 3 "" H 6700 3300 60  0001 C CNN
 F 4 "Stackpole" H 8050 7800 60  0001 C CNN "Mfg"
@@
 F 0 "R316" V 6750 3500 50  0000 C CNN
 F 1 "10k" V 6870 3500 50  0000 C CNN
-F 2 "RESC1608x55N" H 6800 3500 60  0001 C CNN
+F 2 "m_cramps:RESC1608x55N" H 6800 3500 60  0001 C CNN
 F 3 "" H 6800 3500 60  0001 C CNN
 F 4 "Stackpole" H 8150 8000 60  0001 C CNN "Mfg"
@@
 F 0 "R308" V 5250 1800 50  0000 C CNN
 F 1 "10k" V 5370 1800 50  0000 C CNN
-F 2 "RESC1608x55N" H 5300 1800 60  0001 C CNN
+F 2 "m_cramps:RESC1608x55N" H 5300 1800 60  0001 C CNN
 F 3 "" H 5300 1800 60  0001 C CNN
 F 4 "Stackpole" H 6650 6300 60  0001 C CNN "Mfg"
@@
 F 0 "R306" V 3450 6700 50  0000 C CNN
 F 1 "4k7" V 3570 6700 50  0000 C CNN
-F 2 "RESC1608x55N" H 3500 6700 60  0001 C CNN
+F 2 "m_cramps:RESC1608x55N" H 3500 6700 60  0001 C CNN
 F 3 "" H 3500 6700 60  0001 C CNN
 F 4 "Stackpole" H 7050 8900 60  0001 C CNN "Mfg"
@@
 F 0 "R307" V 3650 6700 50  0000 C CNN
 F 1 "4k7" V 3770 6700 50  0000 C CNN
-F 2 "RESC1608x55N" H 3700 6700 60  0001 C CNN
+F 2 "m_cramps:RESC1608x55N" H 3700 6700 60  0001 C CNN
 F 3 "" H 3700 6700 60  0001 C CNN
 F 4 "Stackpole" H 7250 8900 60  0001 C CNN "Mfg"
@@
 F 0 "P304" H 7050 6400 60  0000 C CNN
 F 1 "HEADER_3X2" H 7050 6000 60  0001 C CNN
-F 2 "pin_strip_3x2" H 7050 6200 60  0001 C CNN
+F 2 "w_pin_strip:pin_strip_3x2" H 7050 6200 60  0001 C CNN
 F 3 "" H 7050 6200 60  0000 C CNN
 F 4 "Harwin" H 7050 6200 60  0001 C CNN "Mfg"
@@
 F 0 "S301" H 4200 5150 60  0000 C CNN
 F 1 "SHUNT" H 4200 4950 60  0000 C CNN
-F 2 "Shunt" H 4200 5050 60  0001 C CNN
+F 2 "m_cramps:Shunt" H 4200 5050 60  0001 C CNN
 F 3 "" H 4200 5050 60  0000 C CNN
 F 4 "TE" H 9200 3150 60  0001 C CNN "Mfg"
@@
 F 0 "Q305" H 2950 3850 70  0000 C CNN
 F 1 "2N7002K" H 2900 3500 60  0000 C CNN
-F 2 "SOT23GDS" H 3150 3700 60  0001 C CNN
+F 2 "Tinkerforge:SOT23GDS" H 3150 3700 60  0001 C CNN
 F 3 "" H 3150 3700 60  0000 C CNN
 F 4 "Diodes Inc." H 8100 4800 60  0001 C CNN "Mfg"
