File: CRAMPS/steppers.sch (KiCad schematic (older format))
At the start: 55 parts, among them P201 PT_2,5-2-5,0-H, P202 KK-2.54-4W, P203 KK-2.54-4W, P204 KK-2.54-4W, P205 KK-2.54-4W, P206 KK-2.54-4W, P207 KK-2.54-4W, P208 POLOLU_SOCKET, P209 POLOLU_SOCKET, P210 POLOLU_SOCKET, P211 POLOLU_SOCKET, U201 Pololu, U202 Pololu, U203 Pololu, U204 Pololu, U205 Pololu, U206 Pololu

Commit message: Updated schematic for new Kicad
Parts:
- C201, C202, C203, C204, C205, C206: symbol CP1 -> CP1-RESCUE-CRAMPS
- JP201, JP202, JP203, JP204, JP205, JP206: symbol HEADER_3X2 -> HEADER_3x2
- P208, P209, P210, P211: symbol POLOLU_SOCKET -> Pololu_Socket
- S201, S202, S203, S204, S205, S206, S207, S208, S209, S210, S211, S212, S213, S214, S215, S216, S217, S218: symbol SHUNT -> Shunt
- U201, U202, U203, U204, U205, U206: symbol SM_DRIVER -> SM_Driver
Changed lines of the file:
@@
 EESchema Schematic File Version 2
+LIBS:CRAMPS-rescue
 LIBS:power
 LIBS:m_cramps
@@
 LIBS:memory
 LIBS:xilinx
-LIBS:special
 LIBS:microcontrollers
 LIBS:dsp
@@
 LIBS:beagleboneblack
 LIBS:CRAMPS-cache
-EELAYER 27 0
+EELAYER 25 0
 EELAYER END
 $Descr A 11000 8500
@@
 $EndComp
 $Comp
-L CP1 C201
+L CP1-RESCUE-CRAMPS C201
 U 1 1 50FC3200
 P 4200 1750
@@
 	3300 1900 3700 1900
 $Comp
-L HEADER_3X2 JP201
+L HEADER_3x2 JP201
 U 1 1 53289F71
 P 1600 1900
@@
 $EndComp
 $Comp
-L CP1 C202
+L CP1-RESCUE-CRAMPS C202
 U 1 1 5328A20D
 P 4200 3550
@@
 	3300 3700 3700 3700
 $Comp
-L HEADER_3X2 JP202
+L HEADER_3x2 JP202
 U 1 1 5328A227
 P 1600 3700
@@
 $EndComp
 $Comp
-L CP1 C203
+L CP1-RESCUE-CRAMPS C203
 U 1 1 5328A29A
 P 4200 5350
@@
 	3300 5500 3700 5500
 $Comp
-L HEADER_3X2 JP203
+L HEADER_3x2 JP203
 U 1 1 5328A2B4
 P 1600 5500
@@
 $EndComp
 $Comp
-L CP1 C204
+L CP1-RESCUE-CRAMPS C204
 U 1 1 5328A63F
 P 8000 1750
@@
 	7100 1900 7500 1900
 $Comp
-L HEADER_3X2 JP204
+L HEADER_3x2 JP204
 U 1 1 5328A659
 P 5400 1900
@@
 $EndComp
 $Comp
-L CP1 C205
+L CP1-RESCUE-CRAMPS C205
 U 1 1 5328A69E
 P 8000 3550
@@
 	7100 3700 7500 3700
 $Comp
-L HEADER_3X2 JP205
+L HEADER_3x2 JP205
 U 1 1 5328A6B8
 P 5400 3700
@@
 $EndComp
 $Comp
-L CP1 C206
+L CP1-RESCUE-CRAMPS C206
 U 1 1 5328A6FD
 P 8000 5350
@@
 	7100 5500 7500 5500
 $Comp
-L HEADER_3X2 JP206
+L HEADER_3x2 JP206
 U 1 1 5328A717
 P 5400 5500
@@
 	7100 5900 7100 6150
 $Comp
-L SM_DRIVER U201
+L SM_Driver U201
 U 1 1 53302CEC
 P 2750 1800
@@
 $EndComp
 $Comp
-L SM_DRIVER U202
+L SM_Driver U202
 U 1 1 53302D00
 P 2750 3600
@@
 $EndComp
 $Comp
-L SM_DRIVER U204
+L SM_Driver U204
 U 1 1 53302D14
 P 6550 1800
@@
 $EndComp
 $Comp
-L SM_DRIVER U205
+L SM_Driver U205
 U 1 1 53302D28
 P 6550 3600
@@
 $EndComp
 $Comp
-L SM_DRIVER U203
+L SM_Driver U203
 U 1 1 53302D3C
 P 2750 5400
@@
 $EndComp
 $Comp
-L SM_DRIVER U206
+L SM_Driver U206
 U 1 1 53302D50
 P 6550 5400
@@
 	3150 7100 3150 7200
 $Comp
-L POLOLU_SOCKET P208
+L Pololu_Socket P208
 U 1 1 535FFA9B
 P 9200 5250
@@
 $EndComp
 $Comp
-L POLOLU_SOCKET P209
+L Pololu_Socket P209
 U 1 1 535FFAAA
 P 9200 6050
@@
 $EndComp
 $Comp
-L POLOLU_SOCKET P210
+L Pololu_Socket P210
 U 1 1 535FFAB9
 P 10100 5250
@@
 $EndComp
 $Comp
-L POLOLU_SOCKET P211
+L Pololu_Socket P211
 U 1 1 535FFAC8
 P 10100 6050
@@
 $EndComp
 $Comp
-L SHUNT S201
+L Shunt S201
 U 1 1 5361767A
 P 9200 2450
@@
 $EndComp
 $Comp
-L SHUNT S202
+L Shunt S202
 U 1 1 53617687
 P 9200 2750
@@
 $EndComp
 $Comp
-L SHUNT S203
+L Shunt S203
 U 1 1 53617698
 P 9200 3050
@@
 $EndComp
 $Comp
-L SHUNT S204
+L Shunt S204
 U 1 1 5361769E
 P 9200 3350
@@
 $EndComp
 $Comp
-L SHUNT S205
+L Shunt S205
 U 1 1 536176A4
 P 9200 3650
@@
 $EndComp
 $Comp
-L SHUNT S206
+L Shunt S206
 U 1 1 536176AA
 P 9200 3950
@@
 $EndComp
 $Comp
-L SHUNT S207
+L Shunt S207
 U 1 1 536176DE
 P 9600 2450
@@
 $EndComp
 $Comp
-L SHUNT S208
+L Shunt S208
 U 1 1 536176E4
 P 9600 2750
@@
 $EndComp
 $Comp
-L SHUNT S209
+L Shunt S209
 U 1 1 536176EA
 P 9600 3050
@@
 $EndComp
 $Comp
-L SHUNT S210
+L Shunt S210
 U 1 1 536176F0
 P 9600 3350
@@
 $EndComp
 $Comp
-L SHUNT S211
+L Shunt S211
 U 1 1 536176F6
 P 9600 3650
@@
 $EndComp
 $Comp
-L SHUNT S212
+L Shunt S212
 U 1 1 536176FC
 P 9600 3950
@@
 $EndComp
 $Comp
-L SHUNT S213
+L Shunt S213
 U 1 1 53617702
 P 10000 2450
@@
 $EndComp
 $Comp
-L SHUNT S214
+L Shunt S214
 U 1 1 53617708
 P 10000 2750
@@
 $EndComp
 $Comp
-L SHUNT S215
+L Shunt S215
 U 1 1 5361770E
 P 10000 3050
@@
 $EndComp
 $Comp
-L SHUNT S216
+L Shunt S216
 U 1 1 53617714
 P 10000 3350
@@
 $EndComp
 $Comp
-L SHUNT S217
+L Shunt S217
 U 1 1 5361771A
 P 10000 3650
@@
 $EndComp
 $Comp
-L SHUNT S218
+L Shunt S218
 U 1 1 53617720
 P 10000 3950

Commit message: Fixed the pcb associations in the schematic
Parts:
- C201, C202, C203, C204, C205, C206: footprint c_elec_6.3x7.7 -> Capacitors_SMD:c_elec_6.3x7.7
- F201: footprint Fuse-Loose -> m_cramps:Fuse-Loose
- FH201: footprint Keystone-3568 -> m_cramps:Keystone-3568
- JP201, JP202, JP203, JP204, JP205, JP206: footprint pin_strip_3x2 -> w_pin_strip:pin_strip_3x2
- P201: footprint PT_2,5-2-5,0-H -> m_cramps:PT_2,5-2-5,0-H
- P202, P203, P204, P205, P206, P207: footprint CONN_KK_2.54_4W -> RMC:CONN_KK_2.54_4W
- P208, P209, P210, P211: footprint Pololu_Socket -> m_cramps:Pololu_Socket
- R201, R202, R203, R204, R205, R206: footprint RESC1608x55N -> m_cramps:RESC1608x55N
- S201, S202, S203, S204, S205, S206, S207, S208, S209, S210, S211, S212, S213, S214, S215, S216, S217, S218: footprint Shunt -> m_cramps:Shunt
- U201, U202, U203, U204, U205, U206: footprint POLOLU -> m_cramps:POLOLU
